Commit message: jetbot ready

File: project2/jetbot/urdf/jetbot_rviz.xacro (robot description, xacro)
@@ -3,9 +3,9 @@
     <xacro:include filename="$(find jetbot)/urdf/jetbot.gazebo" />
     <!-- Used for fixing robot to Gazebo 'base_link' -->
-    <link name="world"/>
-    <joint name="fixed" type="fixed">
+    <!-- <link name="world"/> -->
+    <!-- <joint name="fixed" type="fixed">
       <parent link="world"/>
       <child link="chassis"/>
-    </joint>
+    </joint> -->
     <link name="chassis">
       <inertial>
@@ -27,4 +27,80 @@
       </visual>
     </link>
+  <link
+    name="base_laser">
+    <inertial>
+      <origin
+        xyz="-0.00029774 0.0066667 0.00013047"
+        rpy="0 0 0" />
+      <mass
+        value="0.15717" />
+      <inertia
+        ixx="6.7885E-05"
+        ixy="-1.3987E-07"
+        ixz="-8.1554E-07"
+        iyy="0.00013173"
+        iyz="-9.0932E-08"
+        izz="7.1972E-05" />
+    </inertial>
+    <visual>
+        <origin rpy="0.0 0.0 0.0" xyz="0.0 0.0 0"/>
+      <geometry>
+        <mesh
+          filename="file://$(find jetbot)/meshes/ydlidar.dae" />
+      </geometry>
+      <material
+        name="">
+        <color
+          rgba="0.64706 0.61961 0.58824 1" />
+      </material>
+    </visual>
+    <collision>
+        <origin rpy="0.0 0.0 0.0" xyz="0.0 0.0 0"/>
+      <geometry>
+        <mesh
+          filename="file://$(find jetbot)/meshes/ydlidar.dae" />
+      </geometry>
+    </collision>
+  </link>
+<link name='lidarBase'>
+    <pose>0 0 0.1 0 0 0</pose>
+    <inertial>
+      <mass value="1.0"/>
+      <origin xyz="0.0 0 0" rpy=" 0 0 0"/>
+      <inertia
+          ixx="0.1" ixy="0" ixz="0"
+          iyy="0.1" iyz="0"
+          izz="0.1"
+      />
+    </inertial>
+    <collision name='collision'>
+      <origin xyz="0 0 0" rpy=" 0 0 0"/>
+      <geometry>
+        <box size=".18 .13 .01"/>
+      </geometry>
+    </collision>
+    <visual name='visual'>
+      <origin xyz="0 0 0" rpy=" 0 0 0"/>
+      <geometry>
+        <box size=".18 .13 .01" />
+      </geometry>
+    </visual>
+</link>
+<joint type="fixed" name="lidarBase_Joint">
+ <origin xyz="0.0 0 0.2" rpy="0 0 0"/>
+ <child link="lidarBase"/>
+ <parent link="chassis"/>
+ <axis xyz="0 0 1" rpy="0 0 0"/>
+ <limit effort="10000" velocity="1000"/>
+ <dynamics damping="1.0" friction="1.0"/>
+</joint>
+<joint type="fixed" name="base_laser_joint">
+ <origin xyz="0.0 0 0.205" rpy="0 0 0"/>
+ <child link="base_laser"/>
+ <parent link="chassis"/>
+ <axis xyz="0 0 1" rpy="0 0 0"/>
+ <limit effort="10000" velocity="1000"/>
+ <dynamics damping="1.0" friction="1.0"/>
+</joint>
     <link name="left_wheel">
       <inertial>
@@ -81,5 +157,5 @@
     <joint name="camera_joint" type="fixed">
       <origin rpy="0 0.25 0" xyz="0.11 0.0 0.1714"/>
-      <child  link="camera_link"/>
+      <child  link="camera"/>
       <parent link="chassis"/>
       <pose>0.0 0.0 0.0 0.0 0.0 0.0</pose>
@@ -89,5 +165,5 @@
     </joint>
     <!-- Camera -->
-    <link name="camera_link">
+    <link name="camera">
       <gravity>false</gravity>
       <inertial>
@@ -106,5 +182,5 @@
           won't be aligned properly with the frame it is supposedly originating from -->
       <origin xyz="0 0 0" rpy="0 0 0"/>
-      <parent link="camera_link"/>
+      <parent link="camera"/>
       <child link="camera_link_optical"/>
     </joint>
