Commit message: Update jetbot_rviz.xacro

File: whereAmI/jetbot/urdf/jetbot_rviz.xacro (robot description, xacro)
@@ -10,5 +10,5 @@
     <link name="chassis">
       <inertial>
-        <mass value="2.0"/>
+        <mass value="15.0"/>
         <origin rpy="0 0 0" xyz="0 0 0"/>
         <inertia ixx="0.08025" ixy="0" ixz="0" iyy="0.08025" iyz="0" izz="0.1445"/>
@@ -66,5 +66,5 @@
     <pose>0 0 0.1 0 0 0</pose>
     <inertial>
-      <mass value="1.0"/>
+      <mass value="2.0"/>
       <origin xyz="0.0 0 0" rpy=" 0 0 0"/>
       <inertia
@@ -105,5 +105,5 @@
     <link name="left_wheel">
       <inertial>
-        <mass value="0.3"/>
+        <mass value="5"/>
         <origin rpy="0 0 0" xyz="0 0 0"/>
         <inertia ixx="0.000129167" ixy="0" ixz="0" iyy="0.000129167" iyz="0" izz="0.0000225"/>
@@ -131,5 +131,5 @@
     <link name="right_wheel">
       <inertial>
-        <mass value="0.3"/>
+        <mass value="5"/>
         <origin rpy="0 0 0" xyz="0 0 0"/>
         <inertia ixx="0.000129167" ixy="0" ixz="0" iyy="0.000129167" iyz="0" izz="0.0000225"/>

Commit message: Update jetbot_rviz.xacro

File: whereAmI/jetbot/urdf/jetbot_rviz.xacro (robot description, xacro)
@@ -122,5 +122,5 @@
       </visual>
     </link>
-    <joint name='left_wheel_hinge' type='revolute'>
+    <joint name='left_wheel_hinge' type='continuous'>
       <origin rpy="0.0 0.0 1.57079632679" xyz="0.06 0.1025 0.06"/>
       <child  link="left_wheel"/>
@@ -148,5 +148,5 @@
       </visual>
     </link>
-    <joint name='right_wheel_hinge' type='revolute'>
+    <joint name='right_wheel_hinge' type='continuous'>
       <origin rpy="0.0 0.0 1.57079632679 " xyz="0.06 -0.119 0.06"/>
       <child  link="right_wheel"/>

Commit message: updated amcl

File: whereAmI/jetbot/urdf/jetbot_rviz.xacro (robot description, xacro)
@@ -10,5 +10,5 @@
     <link name="chassis">
       <inertial>
-        <mass value="2.0"/>
+        <mass value="15.0"/>
         <origin rpy="0 0 0" xyz="0 0 0"/>
         <inertia ixx="0.08025" ixy="0" ixz="0" iyy="0.08025" iyz="0" izz="0.1445"/>
@@ -105,5 +105,5 @@
     <link name="left_wheel">
       <inertial>
-        <mass value="0.3"/>
+        <mass value="5"/>
         <origin rpy="0 0 0" xyz="0 0 0"/>
         <inertia ixx="0.000129167" ixy="0" ixz="0" iyy="0.000129167" iyz="0" izz="0.0000225"/>
@@ -122,5 +122,5 @@
       </visual>
     </link>
-    <joint name='left_wheel_hinge' type='revolute'>
+    <joint name='left_wheel_hinge' type='continuous'>
       <origin rpy="0.0 0.0 1.57079632679" xyz="0.06 0.1025 0.06"/>
       <child  link="left_wheel"/>
@@ -131,5 +131,5 @@
     <link name="right_wheel">
       <inertial>
-        <mass value="0.3"/>
+        <mass value="5"/>
         <origin rpy="0 0 0" xyz="0 0 0"/>
         <inertia ixx="0.000129167" ixy="0" ixz="0" iyy="0.000129167" iyz="0" izz="0.0000225"/>
@@ -148,5 +148,5 @@
       </visual>
     </link>
-    <joint name='right_wheel_hinge' type='revolute'>
+    <joint name='right_wheel_hinge' type='continuous'>
       <origin rpy="0.0 0.0 1.57079632679 " xyz="0.06 -0.119 0.06"/>
       <child  link="right_wheel"/>
